File: lir2450-charger/lir2450-charger.sch (KiCad schematic (older format))
At the start: 10 parts, among them P1 USB_C_Plug_USB2.0, U1 MCP73831-2-OT

Commit message: Adds green led & pcb icons
Parts:
- added D2: Green LED, LED_SMD:LED_0805_2012Metric, symbol Device:LED
- added R5: 220, Resistor_SMD:R_0805_2012Metric, symbol Device:R_Small_US
- D1: value LED -> Red LED
- R2: value 470 -> 220
Connections:
- net GND: now also D2.1 (K)
- net at R2.2, U1.1 (STAT): now also R5.1
- new net: D2.2 (A), R5.2
Changed lines of the file:
@@
 EESchema Schematic File Version 4
+LIBS:lir2450-charger-cache
 EELAYER 29 0
 EELAYER END
@@
 P 3925 3250
 F 0 "D1" V 3964 3133 50  0000 R CNN
-F 1 "LED" V 3873 3133 50  0000 R CNN
+F 1 "Red LED" V 3873 3133 50  0000 R CNN
 F 2 "LED_SMD:LED_0805_2012Metric" H 3925 3250 50  0001 C CNN
 F 3 "~" H 3925 3250 50  0001 C CNN
@@
 P 3925 3650
 F 0 "R2" H 4050 3725 50  0000 L CNN
-F 1 "470" H 4050 3625 50  0000 L CNN
+F 1 "220" H 4050 3625 50  0000 L CNN
 F 2 "Resistor_SMD:R_0805_2012Metric" H 3925 3650 50  0001 C CNN
 F 3 "~" H 3925 3650 50  0001 C CNN
@@
 	1    0    0    -1
 $EndComp
+$Comp
+L Device:R_Small_US R5
+U 1 1 601054D3
+P 3925 4050
+F 0 "R5" H 4050 4125 50  0000 L CNN
+F 1 "220" H 4050 4025 50  0000 L CNN
+F 2 "Resistor_SMD:R_0805_2012Metric" H 3925 4050 50  0001 C CNN
+F 3 "~" H 3925 4050 50  0001 C CNN
+	1    3925 4050
+	1    0    0    -1
+$EndComp
+$Comp
+L Device:LED D2
+U 1 1 60105912
+P 3925 4400
+F 0 "D2" V 3964 4283 50  0000 R CNN
+F 1 "Green LED" V 3873 4283 50  0000 R CNN
+F 2 "LED_SMD:LED_0805_2012Metric" H 3925 4400 50  0001 C CNN
+F 3 "~" H 3925 4400 50  0001 C CNN
+	1    3925 4400
+	0    -1   -1   0
+$EndComp
+Wire Wire Line
+	3925 3850 3925 3950
+Connection ~ 3925 3850
+Wire Wire Line
+	3925 4150 3925 4250
+$Comp
+L power:GND #PWR0109
+U 1 1 60107677
+P 3925 4650
+F 0 "#PWR0109" H 3925 4400 50  0001 C CNN
+F 1 "GND" H 3930 4477 50  0000 C CNN
+F 2 "" H 3925 4650 50  0001 C CNN
+F 3 "" H 3925 4650 50  0001 C CNN
+	1    3925 4650
+	1    0    0    -1
+$EndComp
+Wire Wire Line
+	3925 4550 3925 4650
 $EndSCHEMATC

Commit message: Adds proper battery footprint
Parts:
- BAT1: footprint Battery:BatteryHolder_Keystone_3008_1x2450 -> Footprints:BatteryHolder_Keystone_3008_1x2450
Changed lines of the file:
@@
 F 0 "BAT1" H 4728 2678 60  0000 L CNN
 F 1 "BS-7" H 4728 2572 60  0000 L CNN
-F 2 "Battery:BatteryHolder_Keystone_3008_1x2450" H 4800 2825 60  0001 L CNN
+F 2 "Footprints:BatteryHolder_Keystone_3008_1x2450" H 4800 2825 60  0001 L CNN
 F 3 "http://www.memoryprotectiondevices.com/datasheets/BS-7-datasheet.pdf" V 4800 2925 60  0001 L CNN
 F 4 "BS-7-ND" H 4800 3025 60  0001 L CNN "Digi-Key_PN"

Commit message: Updates R2 and R5 to 1k
Parts:
- R2, R5: value 220 -> 1k
Changed lines of the file:
@@
 P 3925 3650
 F 0 "R2" H 4050 3725 50  0000 L CNN
-F 1 "220" H 4050 3625 50  0000 L CNN
+F 1 "1k" H 4050 3625 50  0000 L CNN
 F 2 "Resistor_SMD:R_0805_2012Metric" H 3925 3650 50  0001 C CNN
 F 3 "~" H 3925 3650 50  0001 C CNN
@@
 P 3925 4050
 F 0 "R5" H 4050 4125 50  0000 L CNN
-F 1 "220" H 4050 4025 50  0000 L CNN
+F 1 "1k" H 4050 4025 50  0000 L CNN
 F 2 "Resistor_SMD:R_0805_2012Metric" H 3925 4050 50  0001 C CNN
 F 3 "~" H 3925 4050 50  0001 C CNN
